File: ai03_tutorial/_saved_ai03_tutorial.sch (KiCad schematic (older format))
At the start: 24 parts, among them SW1 SW_Push, U1 ATmega32U4-AU, Y1 16Mhz

Commit message: First version of PCB
Parts:
- gave numbers to parts that had none: 1
Changed lines of the file:
@@
 $EndComp
 $Comp
-L Device:C_Small C?
+L Device:C_Small C3
 U 1 1 5C669A95
 P 4250 2250
-F 0 "C?" V 4479 2250 50  0000 C CNN
+F 0 "C3" V 4479 2250 50  0000 C CNN
 F 1 "22pF" V 4388 2250 50  0000 C CNN
 F 2 "Capacitors_SMD:C_0805" H 4250 2250 50  0001 C CNN
